File: Taz Main PCB V1.14.kicad_pcb (KiCad board)
At the start: 4 copper layers, 59.5 x 117 mm, 113 parts, among them CN1 Solar Panel, CN2 Auxilary Conn, CN3 Aux Conn 2, CN4 APCI0136-P001A, CN5 RS232 Conn, J1 Screw_Terminal_01x01, Q1 AO4459, Q2 IRLML6244, SW1 500ASSP1M6QE, SW2 Telemitry Switch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

Commit message: Updated with PDF
Routing:
- net GND: track 261.0 -> 270.2 mm
Changed lines of the file:
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@@
     (pad_to_mask_clearance 0)
     (pcbplotparams
-      (layerselection 0x0000000_fffffff8)
-      (plot_on_all_layers_selection 0x0001055_80000000)
+      (layerselection 0x0000000_7ffffffc)
+      (plot_on_all_layers_selection 0x00010cf_00000004)
       (disableapertmacros false)
       (usegerberextensions false)
@@
   (segment (start 137.75 129.2) (end 137.75 127.75) (width 0.25) (layer "B.Cu") (net 2))
   (segment (start 147.475 105.25) (end 156.625 105.25) (width 0.5) (layer "B.Cu") (net 2))
+  (segment (start 150.1 50.6) (end 151.2625 50.6) (width 0.15) (layer "B.Cu") (net 2))
   (segment (start 171.5 77.25) (end 171 77.25) (width 0.75) (layer "B.Cu") (net 2))
   (segment (start 159.5 104.25) (end 159.5 107.575) (width 0.25) (layer "B.Cu") (net 2))
+  (segment (start 150.25 52) (end 150.45 51.8) (width 0.15) (layer "B.Cu") (net 2))
   (segment (start 143.525 129.175) (end 143.5 129.2) (width 0.25) (layer "B.Cu") (net 2))
   (segment (start 135.3875 138.475) (end 136.475 138.475) (width 0.25) (layer "B.Cu") (net 2))
@@
   (segment (start 160 96.1) (end 163.375 96.1) (width 0.25) (layer "B.Cu") (net 2))
   (segment (start 159.5 104.25) (end 159.5 102.925) (width 0.25) (layer "B.Cu") (net 2))
+  (segment (start 149.5 50) (end 150.1 50.6) (width 0.15) (layer "B.Cu") (net 2))
   (segment (start 176.75 108.25) (end 171.05 108.25) (width 1) (layer "B.Cu") (net 2))
   (segment (start 142.8 53.1875) (end 142.8 55.3) (width 0.25) (layer "B.Cu") (net 2))
@@
   (segment (start 148.5 54.5) (end 148.5 55.25) (width 0.5) (layer "B.Cu") (net 2))
   (segment (start 145 151.25) (end 145 152.5) (width 0.25) (layer "B.Cu") (net 2))
+  (segment (start 150.25 52.5) (end 150.25 52) (width 0.15) (layer "B.Cu") (net 2))
   (segment (start 159.5 102.925) (end 159.05 102.475) (width 0.25) (layer "B.Cu") (net 2))
   (segment (start 164.225 95.25) (end 165.5 95.25) (width 0.25) (layer "B.Cu") (net 2))
   (segment (start 144.5 150.75) (end 145 151.25) (width 0.25) (layer "B.Cu") (net 2))
+  (segment (start 151.2625 53.5125) (end 151.2625 52.2) (width 0.15) (layer "B.Cu") (net 2))
   (segment (start 173.75 78.5) (end 172.5 79.75) (width 0.75) (layer "B.Cu") (net 2))
   (segment (start 173.75 59.5) (end 173.75 75) (width 0.75) (layer "B.Cu") (net 2))
@@
   (segment (start 143.25 128.95) (end 143.5 129.2) (width 0.25) (layer "B.Cu") (net 2))
   (segment (start 159.5 107.575) (end 159.05 108.025) (width 0.25) (layer "B.Cu") (net 2))
+  (segment (start 152.625 54.625) (end 152.375 54.625) (width 0.15) (layer "B.Cu") (net 2))
   (segment (start 131.5 140) (end 131.625 140.125) (width 0.25) (layer "B.Cu") (net 2))
   (segment (start 143 90.75) (end 143.25 90.75) (width 0.25) (layer "B.Cu") (net 2))
+  (segment (start 150.45 51.8) (end 151.2625 51.8) (width 0.15) (layer "B.Cu") (net 2))
   (segment (start 148.75 92.525) (end 148.75 95.475) (width 0.25) (layer "B.Cu") (net 2))
   (segment (start 137.25 140.25) (end 137 140.5) (width 0.25) (layer "B.Cu") (net 2))
+  (segment (start 151.375 53.625) (end 151.2625 53.5125) (width 0.15) (layer "B.Cu") (net 2))
   (segment (start 146.75 133.2) (end 146.75 131) (width 0.25) (layer "B.Cu") (net 2))
   (segment (start 145 152.75) (end 144.5 153.25) (width 0.25) (layer "B.Cu") (net 2))
@@
   (segment (start 137.25 139.25) (end 137.25 139.5) (width 0.25) (layer "B.Cu") (net 2))
   (segment (start 173.75 75) (end 173.75 78.5) (width 0.75) (layer "B.Cu") (net 2))
+  (segment (start 152.375 54.625) (end 151.375 53.625) (width 0.15) (layer "B.Cu") (net 2))
   (segment (start 132.25 140.55) (end 132.05 140.55) (width 0.25) (layer "B.Cu") (net 2))
+  (segment (start 153.25 55.25) (end 152.625 54.625) (width 0.15) (layer "B.Cu") (net 2))
   (segment (start 173.75 75) (end 171.5 77.25) (width 0.75) (layer "B.Cu") (net 2))
+  (segment (start 151.375 53.625) (end 150.25 52.5) (width 0.15) (layer "B.Cu") (net 2))
   (segment (start 163.5 95.975) (end 164.225 95.25) (width 0.25) (layer "B.Cu") (net 2))
   (segment (start 137 140.5) (end 136.95 140.55) (width 0.25) (layer "B.Cu") (net 2))
@@
   (segment (start 154.2875 52.25) (end 154.2375 52.2) (width 0.15) (layer "B.Cu") (net 118))
   (segment (start 161.25 49.5) (end 158.75 47) (width 1) (layer "B.Cu") (net 118))
-  (segment (start 150.35 51.4) (end 151.2625 51.4) (width 0.15) (layer "B.Cu") (net 119))
-  (segment (start 151.75 53.75) (end 151.25 53.25) (width 0.15) (layer "B.Cu") (net 119))
-  (segment (start 151.75 55.75) (end 151.75 53.75) (width 0.15) (layer "B.Cu") (net 119))
-  (segment (start 160.75 56) (end 159 56) (width 0.15) (layer "B.Cu") (net 119))
-  (segment (start 150 53) (end 150 51.75) (width 0.15) (layer "B.Cu") (net 119))
+  (segment (start 151.75 55.75) (end 151.75 54.75) (width 0.15) (layer "B.Cu") (net 119))
+  (segment (start 157 58) (end 154 58) (width 0.15) (layer "B.Cu") (net 119))
   (segment (start 161 55.0375) (end 161 54.1125) (width 0.15) (layer "B.Cu") (net 119))
+  (segment (start 149.75 52) (end 150.35 51.4) (width 0.15) (layer "B.Cu") (net 119))
+  (segment (start 149.75 52.75) (end 149.75 52) (width 0.15) (layer "B.Cu") (net 119))
   (segment (start 161 55.75) (end 160.75 56) (width 0.15) (layer "B.Cu") (net 119))
-  (segment (start 150.25 53.25) (end 150 53) (width 0.15) (layer "B.Cu") (net 119))
-  (segment (start 157 58) (end 154 58) (width 0.15) (layer "B.Cu") (net 119))
+  (segment (start 154 58) (end 151.75 55.75) (width 0.15) (layer "B.Cu") (net 119))
   (segment (start 161 55.0375) (end 161 55.75) (width 0.15) (layer "B.Cu") (net 119))
-  (segment (start 151.25 53.25) (end 150.25 53.25) (width 0.15) (layer "B.Cu") (net 119))
-  (segment (start 150 51.75) (end 150.35 51.4) (width 0.15) (layer "B.Cu") (net 119))
+  (segment (start 151.75 54.75) (end 149.75 52.75) (width 0.15) (layer "B.Cu") (net 119))
   (segment (start 161.5 55.25) (end 163.750001 55.249999) (width 0.15) (layer "B.Cu") (net 119))
   (segment (start 160.75 56) (end 161.5 55.25) (width 0.15) (layer "B.Cu") (net 119))
-  (segment (start 154 58) (end 151.75 55.75) (width 0.15) (layer "B.Cu") (net 119))
-  (segment (start 163.75 55.25) (end 163.750001 55.249999) (width 0.25) (layer "B.Cu") (net 119))
+  (segment (start 150.35 51.4) (end 151.2625 51.4) (width 0.15) (layer "B.Cu") (net 119))
   (segment (start 159 56) (end 157 58) (width 0.15) (layer "B.Cu") (net 119))
+  (segment (start 160.75 56) (end 159 56) (width 0.15) (layer "B.Cu") (net 119))
+  (segment (start 163.75 55.25) (end 163.750001 55.249999) (width 0.25) (layer "B.Cu") (net 119))
   (segment (start 164 94.35) (end 164 96) (width 0.25) (layer "F.Cu") (net 120))
   (segment (start 161.5 96) (end 161.5 94.4) (width 0.25) (layer "F.Cu") (net 121))
